File: converted/N64.kicad_pcb (KiCad board)
At the start: 2 copper layers, 0 parts

Commit message: Clean up
Parts:
- added 3V3: LM22680, PSOP-8, B.Cu at (158.2, 144.9)
- added @HOLE0: , , F.Cu at (111.0, 70.6)
- added @HOLE1: , , F.Cu at (115.2, 112.9)
- added @HOLE2: , , F.Cu at (149.8, 115.1)
- added @HOLE3: , , F.Cu at (128.2, 151.3)
- added @HOLE4: , , F.Cu at (141.5, 151.3)
- added @HOLE5: , , F.Cu at (94.5, 57.3)
- added @HOLE6: , , F.Cu at (202.5, 57.3)
- added @HOLE7: , , F.Cu at (94.5, 152.5)
- added @HOLE8: , , F.Cu at (202.5, 152.5)
- added @HOLE9: , , F.Cu at (164.8, 72.9)
- added AV: PINHEAD-1X8, 2MMPINHEAD-1X8, F.Cu at (196.8, 82.7)
- added BUTT1: PINHEAD-1X8, 2MMPINHEAD-1X8, F.Cu at (100.3, 78.2)
- added BUTT2: PINHEAD-1X8, 2MMPINHEAD-1X8, F.Cu at (196.8, 122.0)
- added C11: , C0805, B.Cu at (186.6, 89.7)
- added C12: , C0805, B.Cu at (186.6, 85.9)
- added C122: , C0805, B.Cu at (193.0, 103.6)
- added C123: , C0805, B.Cu at (187.2, 151.3)
- added C124: c, C0805, F.Cu at (170.9, 94.7)
- added C125: c, C0805, F.Cu at (170.9, 90.9)
- added C126: c, C0805, F.Cu at (170.9, 86.9)
- added C127: , C0805, F.Cu at (186.0, 119.5)
- added C128: 10uF, C0805, F.Cu at (186.0, 115.7)
- added C13: , C0805, B.Cu at (186.6, 82.0)
- added C132: , C0805, B.Cu at (128.2, 118.2)
- added C14: , C0805, F.Cu at (186.0, 89.7)
- added C143: c, C0805, F.Cu at (165.3, 83.4)
- added C144: , C0805, B.Cu at (156.1, 113.2)
- added C146: , C0805, B.Cu at (172.0, 114.4)
- added C147: , C0805, B.Cu at (172.0, 119.5)
- added C15: 10uF, C0805, F.Cu at (186.0, 82.0)
- added C155: , C0805, B.Cu at (95.2, 93.0)
- added C156: , C0805, B.Cu at (100.9, 104.5)
- added C157: , C0805, B.Cu at (191.1, 140.5)
- added C158: , C0805, B.Cu at (191.1, 146.2)
- added C16: 10uF, C0805, F.Cu at (186.0, 85.9)
- added C21: , C0805, B.Cu at (179.0, 90.9)
- added C23: , C0805, B.Cu at (193.0, 98.6)
- added C24: 10uF, C0805, B.Cu at (178.4, 108.7)
- added C25: 10uF, C0805, F.Cu at (186.0, 99.8)
- added C26: 10uF, C0805, F.Cu at (186.0, 103.6)
- added C28: 10uF, C0805, B.Cu at (178.4, 104.9)
- added C29_X: , C0805, F.Cu at (186.0, 111.9)
- added C30: , C0805, F.Cu at (186.0, 107.4)
- added C31: , C0805, F.Cu at (168.2, 106.2)
- added C32: , C0805, F.Cu at (168.2, 101.7)
- added C33: 68uF, C%2f6032-28R, F.Cu at (158.8, 111.4)
- added C34: 10uF, C0805, B.Cu at (171.4, 108.7)
- added C39: , C0805, B.Cu at (167.6, 127.8)
- added C40_: , C0805, B.Cu at (154.2, 126.5)
- added C5: , C0805K, B.Cu at (105.3, 83.3)
- added C6: , C0805, B.Cu at (105.3, 90.9)
- added C7: , C0805, B.Cu at (105.3, 87.8)
- added C8: , C0805, B.Cu at (105.3, 94.7)
- added C9: , C0805, B.Cu at (105.3, 79.5)
- added CA: , C1206K, B.Cu at (158.2, 138.6)
- added CA1: , C1206K, B.Cu at (154.5, 151.4)
- added CA10: , C0805K, F.Cu at (149.3, 151.1)
- added CA11: , C0805K, B.Cu at (148.1, 150.0)
- added CA12: , C0805K, B.Cu at (168.1, 142.0)
- added CA2: , C0805K, B.Cu at (133.3, 126.5)
- added CA3: , C1210K, F.Cu at (150.8, 139.4)
- added CA4: , C1206K, B.Cu at (149.3, 143.5)
- added CA5: , C0805K, B.Cu at (133.3, 136.0)
- added CA6: 470pF, C0805K, B.Cu at (133.3, 131.6)
- added CA7: , C0805K, B.Cu at (135.2, 154.1)
- added CA8: , C0805K, B.Cu at (140.6, 146.7)
- added CA9: 470pF, C0805K, B.Cu at (130.6, 146.7)
- added CD1: 10uF, C0805, F.Cu at (106.1, 99.7)
- added CD10: 10uF, C0805, B.Cu at (125.7, 65.0)
- added CD11: 10uF, C0805, B.Cu at (129.6, 65.3)
- added CD12: 10uF, C0805, B.Cu at (133.9, 65.7)
- added CD13: 10uF, C0805, B.Cu at (137.0, 65.7)
- added CD14: 10uF, C0805, B.Cu at (144.4, 72.4)
- added CD15: 10uF, C0805, B.Cu at (148.4, 79.5)
- added CD16: 10uF, C0805, B.Cu at (147.9, 82.8)
- added CD17: 10uF, C0805, B.Cu at (147.9, 86.1)
- added CD18: 10uF, C0805, B.Cu at (147.9, 89.4)
- added CD19: 10uF, C0805, B.Cu at (147.9, 92.7)
- added CD2: 10uF, C0805, F.Cu at (106.1, 94.9)
- added CD20: 10uF, C0805, B.Cu at (147.9, 96.0)
- added CD21: 10uF, C0805, B.Cu at (138.4, 108.1)
- added CD22: 10uF, C0805, B.Cu at (133.9, 108.1)
- added CD23: 10uF, C0805, B.Cu at (129.5, 108.1)
- added CD24: 10uF, C0805, B.Cu at (125.0, 108.1)
- added CD25: 10uF, C0805, B.Cu at (120.6, 108.1)
- added CD26: 10uF, C0805, B.Cu at (116.1, 108.0)
- added CD27: 10uF, C0805, B.Cu at (143.8, 107.3)
- added CD28: 10uF, C0805, B.Cu at (147.7, 102.7)
- added CD29: 10uF, C0805, B.Cu at (147.9, 99.4)
- added CD3: 10uF, C0805, F.Cu at (106.3, 87.9)
- added CD30: 10uF, C0805, B.Cu at (147.9, 106.2)
- added CD31: 10uF, C0805, B.Cu at (153.6, 93.5)
- added CD32: 10uF, C0805, B.Cu at (158.4, 97.4)
- added CD33: 10uF, C0805, B.Cu at (153.6, 86.1)
- added CD34: 10uF, C0805, F.Cu at (145.3, 74.8)
- added CD35: 10uF, C0805, F.Cu at (140.3, 76.5)
- added CD36: 10uF, C0805, B.Cu at (158.4, 89.9)
- added CD37: 10uF, C0805, F.Cu at (129.2, 78.1)
- added CD38: 10uF, C0805, F.Cu at (124.6, 78.0)
- added CD39: 10uF, C0805, F.Cu at (117.8, 78.7)
- added CD4: 10uF, C0805, F.Cu at (106.3, 84.2)
- added CD40: 10uF, C0805, F.Cu at (112.3, 84.7)
- added CD41: 10uF, C0805, F.Cu at (112.3, 89.0)
- added CD42: 10uF, C0805, F.Cu at (112.3, 93.5)
- added CD43: 10uF, C0805, F.Cu at (112.3, 96.6)
- added CD44: 10uF, C0805, F.Cu at (112.3, 99.8)
- added CD45: 10uF, C0805, F.Cu at (111.9, 103.0)
- added CD46: 10uF, C0805, F.Cu at (112.3, 106.2)
- added CD47: 10uF, C0805, F.Cu at (112.3, 109.3)
- added CD48: 10uF, C0805, B.Cu at (120.6, 113.2)
- added CD49: 10uF, C0805, B.Cu at (126.2, 113.9)
- added CD5: 10uF, C0805, F.Cu at (106.3, 81.2)
- added CD50: 10uF, C0805, B.Cu at (131.4, 113.9)
- added CD51: 10uF, C0805, B.Cu at (136.7, 113.9)
- added CD52: 10uF, C0805, B.Cu at (140.9, 113.8)
- added CD54: 10uF, C0805, B.Cu at (147.7, 111.3)
- added CD55: 10uF, C0805, F.Cu at (116.8, 131.6)
- added CD56: 10uF, C0805, B.Cu at (179.0, 86.5)
- added CD57: 10uF, C0805, B.Cu at (186.6, 124.0)
- added CD58: 10uF, C0805, B.Cu at (184.7, 146.2)
- added CD59: 10uF, C0805, B.Cu at (178.4, 82.0)
- added CD6: 10uF, C0805, F.Cu at (107.4, 75.2)
- added CD60: 10uF, C0805, F.Cu at (177.1, 92.8)
- added CD61: 10uF, C0805, F.Cu at (178.4, 111.9)
- added CD7: 10uF, C0805, B.Cu at (115.4, 65.7)
- added CD8: 10uF, C0805, B.Cu at (118.3, 65.7)
- added CD9: 10uF, C0805, B.Cu at (122.0, 65.0)
- added CONT1: PINHEAD-1X6, 2MMPINHEAD-1X6, F.Cu at (97.7, 97.9)
- added CONT2: PINHEAD-1X6, 2MMPINHEAD-1X6, F.Cu at (199.3, 142.4)
- added C_C1: , C0805, F.Cu at (107.2, 110.6)
- added C_C14: , C0805, F.Cu at (109.8, 137.3)
- added C_R1: 1M0, M0805, B.Cu at (107.2, 110.6)
- added C_R3: 130R, M0805, F.Cu at (116.8, 137.3)
- added C_R4: 150K, M0805, F.Cu at (109.8, 131.6)
- added C_U1: CNT-NUS, PQFP64, B.Cu at (111.6, 129.3)
- added D1: PMLL4150, SOD80C, B.Cu at (171.4, 104.9)
- added D1: STKYDIODE, STKYDIODE, F.Cu at (158.0, 138.6)
- added D2: PMLL4150, SOD80C, B.Cu at (177.7, 127.8)
- added JOY: PINHEAD-1X6, 2MMPINHEAD-1X6, F.Cu at (199.3, 103.6)
- added JP1: , 1X03, F.Cu at (103.4, 112.5)
- added JP2: , 1X02, F.Cu at (175.7, 151.3)
- added LED1: , CHIPLED_0805, F.Cu at (116.1, 150.0)
- added LED2: , CHIPLED_0805, F.Cu at (116.1, 145.5)
- added LED3: , CHIPLED_0805, F.Cu at (109.1, 150.0)
- added LED4: , CHIPLED_0805, F.Cu at (109.1, 145.5)
- added Q1: , HC49%2fS, F.Cu at (168.2, 117.0)
- added R10: 110R, M0805, B.Cu at (166.7, 86.9)
- added R11: 10k, M0805, F.Cu at (161.7, 82.2)
- added R12: 820R, M0805, B.Cu at (172.6, 90.9)
- added R13: 4k3, M0805, B.Cu at (172.6, 87.1)
- added R17: 1K, M0805, B.Cu at (186.6, 108.1)
- added R18: 10k, M0805, B.Cu at (164.4, 108.7)
- added R19: 180k, M0805, B.Cu at (178.4, 100.5)
- added R2: 2k0, M0805, B.Cu at (171.4, 100.5)
- added R20: 10k, M0805, B.Cu at (164.4, 104.9)
- added R21: 1k, M0805, B.Cu at (186.6, 103.6)
- added R22: 47K, M0805, B.Cu at (186.6, 118.9)
- added R23: 10k, M0805, B.Cu at (186.6, 115.1)
- added R24: 24R, M0805, B.Cu at (146.6, 120.8)
- added R25: 130R, M0805, B.Cu at (135.2, 121.8)
- added R29: 4R7, M0805, B.Cu at (105.3, 75.7)
- added R3: 30K, M0805, F.Cu at (178.4, 115.7)
- added R30: 4R7, M0805, B.Cu at (105.3, 71.9)
- added R32: 150R, M0805, F.Cu at (157.4, 124.6)
- added R33: 33R, M0805, F.Cu at (151.7, 124.6)
- added R34: 47K, M0805, B.Cu at (148.4, 70.1)
- added R35: 390R, M0805, B.Cu at (141.1, 121.8)
- added R36: 51K, M0805, F.Cu at (163.1, 124.6)
- added R37: 750R, M0805, B.Cu at (99.2, 93.0)
- added R38: 750R, M0805, B.Cu at (96.4, 104.5)
- added R39: 750R, M0805, B.Cu at (184.7, 140.5)
- added R4: 68K, M0805, F.Cu at (178.4, 119.5)
- added R40: 750R, M0805, B.Cu at (198.0, 140.5)
- added R5: 75R, M0805, F.Cu at (191.1, 82.0)
- added R53: 130R, M0805, B.Cu at (95.2, 98.2)
- added R54: 130R, M0805, B.Cu at (100.9, 99.4)
- added R55: 130R, M0805, B.Cu at (191.1, 134.1)
- added R56: 130R, M0805, B.Cu at (198.0, 146.2)
- added R57: 1k, M0805, F.Cu at (191.7, 104.3)
- added R58: 1k, M0805, F.Cu at (191.7, 99.8)
- added R6: 75R, M0805, F.Cu at (191.1, 85.9)
- added R7: 75R, M0805, F.Cu at (191.1, 89.7)
- added R8: 110R, M0805, B.Cu at (166.3, 94.7)
- added R9: 110R, M0805, B.Cu at (166.3, 90.9)
- added RA: OPEN, M0805, F.Cu at (109.8, 120.1)
- added RB: 0R, M0805, F.Cu at (116.8, 125.9)
- added RC: 33K, M0805, F.Cu at (109.8, 125.9)
- added RD: 33K, M0805, F.Cu at (116.8, 120.1)
- added RE: 1K4, M0805, B.Cu at (162.4, 151.4)
- added RE1: 1K4, M0805, B.Cu at (116.1, 151.3)
- added RE2: 1K4, M0805, B.Cu at (116.1, 146.8)
- added RE3: 1K4, M0805, B.Cu at (109.1, 151.4)
- added RE4: 1K4, M0805, B.Cu at (109.1, 146.8)
- added RF: 1K0, M0805, B.Cu at (168.3, 151.4)
- added RG: 191k, M0805, B.Cu at (167.9, 146.3)
- added RGB: PINHEAD-1X6, 2MMPINHEAD-1X6, F.Cu at (190.4, 68.1)
- added RN1: RESNET, RESARRAY, B.Cu at (130.7, 142.9)
- added RN2: RESNET, RESARRAY, B.Cu at (137.1, 142.9)
- added RN3: RESNET, RESARRAY, B.Cu at (143.4, 142.9)
- added S1: , B3F-10XX, F.Cu at (187.4, 151.3)
- added TVS1: TVS, SC-74, B.Cu at (199.9, 83.9)
- added TVS2: TVS, SC-74, B.Cu at (184.1, 134.1)
- added TVS3: TVS, SC-74, B.Cu at (98.2, 87.0)
- added TVS4: TVS, SC-74, B.Cu at (197.4, 134.1)
- added TVS5: TVS, SC-74, B.Cu at (99.7, 77.9)
- added TVS6: TVS, SC-74, B.Cu at (197.3, 124.2)
- added U$37: PINHEAD-25X2, PINHEAD-25X2, F.Cu at (146.0, 61.1)
- added U$38: PINHEAD-16X2SMALLER, 2MMPINHEAD-16X2, F.Cu at (100.3, 134.1)
- added U$52: INDUCTOR, INDUCTOR, F.Cu at (159.4, 148.1)
- added U10: R4300_CPU, QFP120, B.Cu at (126.9, 87.1)
- added U11: RDRAM18_NUS, SHP32, F.Cu at (133.9, 141.2)
- added U12: MIC5219, SOT23-5, B.Cu at (135.3, 148.8)
- added U13: MIC5219, SOT23-5, B.Cu at (139.6, 127.8)
- added U14: RDRAM18_NUS, SHP32, F.Cu at (133.9, 123.8)
- added U15: MX8330MC, SO08, F.Cu at (160.6, 131.6)
- added U2: AMP-NUS, SO14, F.Cu at (177.1, 102.4)
- added U3: 9480, SO8, F.Cu at (159.1, 106.2)
- added U3_: U3, SOT23-5, F.Cu at (152.3, 130.3)
- added U4: VDCNUS, SO24, F.Cu at (161.6, 94.6)
- added U5: ENC-NUS, SO14, F.Cu at (174.8, 78.5)
- added U6: PIF, SO28W, F.Cu at (184.1, 132.2)
- added U7: MX8330MC, SO08, F.Cu at (156.8, 117.0)
- added U8: 74LS125J, QSOP14, F.Cu at (177.0, 144.7)
- added U9: N64_RCP, PQFP160, F.Cu at (133.3, 97.3)
- added X2: , HC49%2fS, F.Cu at (171.4, 130.3)
Routing:
- net 3V3: track 0.00 -> 787.2 mm, vias 0 -> 49
- net (no net): track 0.00 -> 242.1 mm, vias 0 -> 79
- net GND: track 0.00 -> 116.9 mm, vias 0 -> 8
- net +12V: track 0.00 -> 97.6 mm, vias 0 -> 2
- net N$161: track 0.00 -> 87.3 mm, vias 0 -> 2
- net N$162: track 0.00 -> 85.5 mm, vias 0 -> 2
- net N$159: track 0.00 -> 83.6 mm, vias 0 -> 2
- net N$7: track 0.00 -> 81.9 mm, vias 0 -> 4
- net N$160: track 0.00 -> 79.9 mm, vias 0 -> 2
- net N$15: track 0.00 -> 75.8 mm, vias 0 -> 2
- net N$163: track 0.00 -> 72.5 mm, vias 0 -> 2
- net /COLDRESET: track 0.00 -> 72.0 mm, vias 0 -> 3
- net NMI: track 0.00 -> 65.4 mm, vias 0 -> 2
- net N$58: track 0.00 -> 49.2 mm, vias 0 -> 2
- net N$51: track 0.00 -> 41.1 mm
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- added copper zone on B.Cu, net 3V3
- added copper zone on F.Cu, net 3V3
- added copper zone on Route15, net 3V3
- added copper zone on B.Cu, net GND
- added copper zone on F.Cu, net GND
Other:
- board outline added: 114.3 x 103.9 mm
- copper layers 2 -> 4
- net class Default: clearance 0.2 -> 0.1524
- rule trace_clearance: 0.2 -> 0.1524
- rule via_min_drill: 0.3 -> 0.2996
- rule via_min_size: 0.4 -> 0.254
- board text removed: "*** THIS IS THE DUMMY SAVE FILE *** IF YOUR ARE READING THIS MESSAGE, YOU HAVE NOT DONE A SAVE-AS IN PCBNEW TO THIS FILE NAME, WHEN IMPORTING A EAGLE PCB FILE TO A KICAD PCB FILE!!"
